Commit message: Simulated the bot in Gazebo

File: my_robot_description/urdf/mobile_base.xacro (robot description, xacro)
@@ -15,4 +15,12 @@
             <material name="blue" />
         </visual>
+        <collision>
+            <geometry>
+                <box size="${base_length} ${base_width} ${base_height}" />
+            </geometry>
+            <origin xyz="0 0 ${base_height / 2.0}" rpy="0 0 0" />
+        </collision>
+        <xacro:box_inertia m="5.0" l="${2*base_length}" w="${2*base_width}" h="${2*base_height}"
+                           xyz="0 0 ${base_height / 2.0}" rpy="0 0 0" />
     </link>
     <xacro:macro name="wheel_link" params="prefix">
@@ -25,4 +33,12 @@
                 <material name="grey" />
             </visual>
+            <collision>
+                <geometry>
+                    <cylinder radius="${wheel_radius}" length="${wheel_length}" />
+                </geometry>
+                <origin xyz="0 0 0" rpy="${pi / 2.0} 0 0" />
+            </collision>
+            <xacro:cylinder_inertia m="1.0" r="${2*wheel_radius}" h="${2*wheel_length}"
+                                    xyz="0 0 0" rpy="${pi / 2.0} 0 0" />
         </link>
     </xacro:macro>
@@ -37,4 +53,12 @@
             <material name="grey" />
         </visual>
+        <collision>
+            <geometry>
+                <sphere radius="${wheel_radius / 2.0}" />
+            </geometry>
+            <origin xyz="0 0 0" rpy="0 0 0" />
+        </collision>
+        <xacro:sphere_inertia m="0.5" r="${2*wheel_radius / 2.0}"
+                              xyz="0 0 0" rpy="0 0 0" />
     </link>
     <joint name="base_joint" type="fixed">

Commit message: Added Camera Sensor

File: my_robot_description/urdf/mobile_base.xacro (robot description, xacro)
@@ -6,5 +6,5 @@
     <xacro:property name="wheel_radius" value="0.1" />
     <xacro:property name="wheel_length" value="0.05" />
-    <link name="base_footprint_link" />
+    <link name="base_footprint" />
     <link name="base_link">
         <visual>
@@ -63,5 +63,5 @@
     </link>
     <joint name="base_joint" type="fixed">
-        <parent link="base_footprint_link" />
+        <parent link="base_footprint" />
         <child link="base_link" />
         <origin xyz="0 0 ${wheel_radius}" rpy="0 0 0"/>

File: my_robot_description/urdf/mobile_base_gazebo.xacro (robot description, xacro)
@@ -31,5 +31,5 @@
             <odometry_topic>odom</odometry_topic>
             <odometry_frame>odom</odometry_frame>
-            <robot_base_frame>base_footprint_link</robot_base_frame>
+            <robot_base_frame>base_footprint</robot_base_frame>
         </plugin>
     </gazebo>

Commit message: Added Ros2-Control and Joystick for motion

File: my_robot_description/urdf/mobile_base.xacro (robot description, xacro)
@@ -35,5 +35,5 @@
             <collision>
                 <geometry>
-                    <cylinder radius="${wheel_radius}" length="${wheel_length}" />
+                    <sphere radius="${wheel_radius}" />
                 </geometry>
                 <origin xyz="0 0 0" rpy="${pi / 2.0} 0 0" />
@@ -63,6 +63,6 @@
     </link>
     <joint name="base_joint" type="fixed">
-        <parent link="base_footprint" />
-        <child link="base_link" />
+        <parent link="base_link" />
+        <child link="base_footprint" />
         <origin xyz="0 0 ${wheel_radius}" rpy="0 0 0"/>
     </joint>

File: my_robot_description/urdf/mobile_base_gazebo.xacro (robot description, xacro)
@@ -15,15 +15,11 @@
         <mu2 value="0.1" />
     </gazebo>
-    <gazebo>
+    <!-- <gazebo>
         <plugin name="diff_drive_controller" filename="libgazebo_ros_diff_drive.so">
-            <!-- Update rate in Hz -->
             <update_rate>50</update_rate>
-            <!-- wheels -->
             <left_joint>base_left_wheel_joint</left_joint>
             <right_joint>base_right_wheel_joint</right_joint>
-            <!-- kinematics -->
             <wheel_separation>0.45</wheel_separation>
             <wheel_diameter>0.2</wheel_diameter>
-            <!-- output -->
             <publish_odom>true</publish_odom>
             <publish_odom_tf>true</publish_odom_tf>
@@ -33,4 +29,31 @@
             <robot_base_frame>base_footprint</robot_base_frame>
         </plugin>
+    </gazebo> -->
+    <ros2_control name="GazeboSystem" type="system">
+        <hardware>
+            <plugin>gazebo_ros2_control/GazeboSystem</plugin>
+        </hardware>
+        <joint name="base_left_wheel_joint">
+            <command_interface name="velocity">
+                <param name="min">-10</param>
+                <param name="max">10</param>
+            </command_interface>
+            <state_interface name="velocity"/>
+            <state_interface name="position"/>
+        </joint>
+        <joint name="base_right_wheel_joint">
+            <command_interface name="velocity">
+                <param name="min">-10</param>
+                <param name="max">10</param>
+            </command_interface>
+            <state_interface name="velocity"/>
+            <state_interface name="position"/>
+        </joint>
+    </ros2_control>
+    <gazebo>
+        <plugin name="gazebo_ros2_control" filename="libgazebo_ros2_control.so">
+            <parameters>$(find my_robot_description)/config/my_controllers.yaml</parameters>
+            <parameters>$(find my_robot_description)/config/gaz_ros2_ctl_use_sim.yaml</parameters>
+        </plugin>
     </gazebo>
 </robot>

File: my_robot_description/urdf/my_robot.urdf.xacro (robot description, xacro)
@@ -6,5 +6,5 @@
     <xacro:include filename="arm.xacro" />
     <xacro:include filename="arm_gazebo.xacro" />
-    <xacro:include filename="camera.xacro" />
+    <!-- <xacro:include filename="camera.xacro" /> -->
     <joint name="mobile_base_arm_joint" type="fixed">
         <parent link="base_link" />
